File: Arduino HomeMonitor.brd (EAGLE design)
At the start: 100 x 100 mm, 28 parts, among them U1 LM358N, U2 DHT22

Commit message: board edit
Routing:
- net S$29: track 0.00 -> 3.58 mm
- net S$20: track 5.38 -> 1.95 mm
Changed lines of the file:
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@@
 </signal>
 <signal name="S$20">
-<wire x1="74.66464375" y1="9.451371875" x2="71.23090625" y2="9.451371875" width="0.4064" layer="16"/>
 <wire x1="71.23090625" y1="9.451371875" x2="69.85135625" y2="10.830921875" width="0.4064" layer="16"/>
 </signal>
@@
 <wire x1="10.892715625" y1="44.447984375" x2="10.746503125" y2="44.301771875" width="0.4064" layer="1"/>
 </signal>
+<signal name="S$28">
+<via x="71.230771875" y="9.480725" extent="1-16" drill="0.5" diameter="0.254"/>
+</signal>
+<signal name="S$29">
+<wire x1="71.260121875" y1="9.42201875" x2="74.75268125" y2="9.42201875" width="0.4064" layer="1"/>
+<wire x1="74.75268125" y1="9.42201875" x2="74.8113875" y2="9.480725" width="0.4064" layer="1"/>
+</signal>
 </signals>
