File: v1/Arduino HomeMonitorv1r4-current.brd (EAGLE design)
At the start: 100 x 100 mm, 34 parts, among them U2 DHT22

Commit message: Rev 4
Fixed some errors
Connections:
- removed net S$172: PD3.2, POWER.2
- net GND: now also PD3.2, POWER.2
Routing:
- net S$24: track 0.00 -> 5.62 mm
- net S$1: track 0.00 -> 5.62 mm
- net S$172: track 2.54 -> 0.00 mm
- net GND: track 296.6 -> 297.9 mm
Other:
- board size 100 x 100 mm -> 83.1 x 58.7 mm
